File: Versions/EyeTrack/1.1/PCBs/MouseGoggles IRLED-1-5/MouseGoggles IRLED-1-5.brd (EAGLE design)
At the start: 20 x 13 mm, 5 parts

Commit message: Update IRLED board
Other:
- board size 20 x 13 mm -> 20 x 13.1 mm
Changed lines of the file:
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@@
 <board>
 <plain>
-<wire x1="0" y1="0.381" x2="4.479290625" y2="0.381" width="0" layer="20"/>
-<wire x1="15.63496875" y1="0.381" x2="19.999959375" y2="0.381" width="0" layer="20"/>
-<wire x1="19.999959375" y1="0.381" x2="19.999959375" y2="13.335" width="0" layer="20"/>
+<wire x1="0" y1="2.032" x2="1.778" y2="0.254" width="0" layer="20"/>
+<wire x1="1.778" y1="0.254" x2="4.479290625" y2="0.254" width="0" layer="20"/>
+<wire x1="15.63496875" y1="0.254" x2="18.161" y2="0.254" width="0" layer="20"/>
+<wire x1="18.161" y1="0.254" x2="19.999959375" y2="2.032" width="0" layer="20"/>
+<wire x1="19.999959375" y1="2.032" x2="19.999959375" y2="13.335" width="0" layer="20"/>
 <wire x1="19.999959375" y1="13.335" x2="0" y2="13.335" width="0" layer="20"/>
-<wire x1="0" y1="13.335" x2="0" y2="0.381" width="0" layer="20"/>
-<wire x1="4.479290625" y1="0.381" x2="4.479290625" y2="9.525" width="0" layer="20"/>
-<wire x1="4.479290625" y1="9.525" x2="15.63496875" y2="9.525" width="0" layer="20"/>
-<wire x1="15.63496875" y1="9.525" x2="15.63496875" y2="0.381" width="0" layer="20"/>
+<wire x1="0" y1="13.335" x2="0" y2="2.032" width="0" layer="20"/>
+<wire x1="4.479290625" y1="0.254" x2="4.479290625" y2="9.652" width="0" layer="20"/>
+<wire x1="4.479290625" y1="9.652" x2="15.63496875" y2="9.652" width="0" layer="20"/>
+<wire x1="15.63496875" y1="9.652" x2="15.63496875" y2="0.254" width="0" layer="20"/>
 </plain>
 <attributes>
